Commit message: feat(serial_port): 新增运行时硬件连接参数覆盖功能

File: src/robot_supports/robots/dm_arm/description/model/gray/urdf/dm_arm.ros2_control.xacro (robot description, xacro)
@@ -4,8 +4,17 @@
     <xacro:arg name="hardware_plugin" default=""/>
     <xacro:arg name="hardware_config" default=""/>
+    <xacro:arg name="serial_port" default=""/>
+    <xacro:arg name="baudrate" default=""/>
+    <xacro:arg name="bus" default=""/>
     <xacro:include filename="$(find dm_arm_description)/model/gray/urdf/dm_arm_no_gripper.urdf"/>
     <xacro:include filename="$(find serial_arm_ros2_control)/urdf/serial_arm_system.ros2_control.xacro"/>
     <ros2_control name="dm_arm" type="system">
-        <xacro:serial_arm_ros2_control_hardware config_file="$(arg config_file)" hardware_plugin="$(arg hardware_plugin)" hardware_config="$(arg hardware_config)"/>
+        <xacro:serial_arm_ros2_control_hardware
+            config_file="$(arg config_file)"
+            hardware_plugin="$(arg hardware_plugin)"
+            hardware_config="$(arg hardware_config)"
+            serial_port="$(arg serial_port)"
+            baudrate="$(arg baudrate)"
+            bus="$(arg bus)"/>
         <joint name="joint1">
             <command_interface name="position"/>

File: src/robot_supports/robots/dm_arm/description/model/white/urdf/dm_arm.ros2_control.xacro (robot description, xacro)
@@ -4,8 +4,17 @@
     <xacro:arg name="hardware_plugin" default=""/>
     <xacro:arg name="hardware_config" default=""/>
+    <xacro:arg name="serial_port" default=""/>
+    <xacro:arg name="baudrate" default=""/>
+    <xacro:arg name="bus" default=""/>
     <xacro:include filename="$(find dm_arm_description)/model/white/urdf/dm_arm.urdf"/>
     <xacro:include filename="$(find serial_arm_ros2_control)/urdf/serial_arm_system.ros2_control.xacro"/>
     <ros2_control name="dm_arm" type="system">
-        <xacro:serial_arm_ros2_control_hardware config_file="$(arg config_file)" hardware_plugin="$(arg hardware_plugin)" hardware_config="$(arg hardware_config)"/>
+        <xacro:serial_arm_ros2_control_hardware
+            config_file="$(arg config_file)"
+            hardware_plugin="$(arg hardware_plugin)"
+            hardware_config="$(arg hardware_config)"
+            serial_port="$(arg serial_port)"
+            baudrate="$(arg baudrate)"
+            bus="$(arg bus)"/>
         <joint name="joint1">
             <command_interface name="position"/>

File: src/serial_arm/bringup/ros2_control/urdf/serial_arm_system.ros2_control.xacro (robot description, xacro)
@@ -1,5 +1,5 @@
 <?xml version="1.0"?>
 <robot xmlns:xacro="http://www.ros.org/wiki/xacro">
-    <xacro:macro name="serial_arm_ros2_control_hardware" params="config_file hardware_plugin hardware_config">
+    <xacro:macro name="serial_arm_ros2_control_hardware" params="config_file hardware_plugin hardware_config serial_port:='' baudrate:='' bus:=''">
         <hardware>
             <plugin>serial_arm_ros2_control/SerialArmSystem</plugin>
@@ -7,4 +7,13 @@
             <param name="hardware_plugin">${hardware_plugin}</param>
             <param name="hardware_config">${hardware_config}</param>
+            <xacro:if value="${serial_port != ''}">
+                <param name="serial_port">${serial_port}</param>
+            </xacro:if>
+            <xacro:if value="${baudrate != ''}">
+                <param name="baudrate">${baudrate}</param>
+            </xacro:if>
+            <xacro:if value="${bus != ''}">
+                <param name="bus">${bus}</param>
+            </xacro:if>
         </hardware>
     </xacro:macro>
