Commit message: fix(calibration): 修复了 urdf 校准算法的计算 bug，测试效果良好，相较于精确称量质量和质心的标定，使用该算法可在不拆卸机械臂的情况下快速完成重力模型校正

File: src/robot_supports/robots/tomato_picker/tomato_picker_description/urdf/tomato_picker.urdf (robot description, URDF)
Before this commit: robot Tomato-Picker, 11 links, 10 joints
Links:
- link Link6: mass 0.785649631359557 -> 0.774251897736

Commit message: perf(gui): 优化标定界面的排版

File: src/robot_supports/robots/tomato_picker/tomato_picker_description/urdf/tomato_picker.urdf (robot description, URDF)
Before this commit: robot Tomato-Picker, 11 links, 10 joints
Links:
- link Link6: mass 0.774251897736 -> 0.785649631359557

Commit message: feat(urdf): 新增 tip link

File: src/robot_supports/robots/tomato_picker/tomato_picker_description/urdf/tomato_picker.urdf (robot description, URDF)
Before this commit: robot Tomato-Picker, 11 links, 10 joints
Links:
- added link tip
Joints:
- added joint tip_joint: type fixed, parent tool0, child tip, origin xyz=0 0 0.101 rpy=0 0 0
